File: Project V2/final project/final project.kicad_pcb (KiCad board)
At the start: 2 copper layers, 77.6 x 23 mm, 46 parts, among them J1 Conn_01x09, J2 Conn_01x12, J3 Conn_01x17, SW1 SW_Push, SW2 SW_Push, U1 CH340C, U2 IP5306, U3 AMS1117, U4 ATmega328P-A, U5 NRF24L01_Breakout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

Commit message: 8/18 update
gerber送廠
Parts:
- added G***: LOGO, LOGO:QR, B.Cu at (98.5, 41.2)
- moved G*** 0.30 mm to (69.0, 41.3)
